File: kicad/power_in_regulator.kicad_sch (KiCad schematic)
At the start: 12 parts, among them U3 AMS1117-3.3, U6 LMR36015ARNXR

Commit message: finish motor driver module
Parts:
- RFBB2: value 24.9k -> 10k
- RFBT2: value 100k -> 52.3k
Changed lines of the file:
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@@
 			)
 		)
-		(property "Value" "100k"
+		(property "Value" "52.3k"
 			(at 174.5635 100.3299 0)
 			(show_name no)
@@
 			)
 		)
-		(property "Value" "24.9k"
+		(property "Value" "10k"
 			(at 174.5635 107.9499 0)
 			(show_name no)

Commit message: edit a lot of stuff
Parts:
- added J2: Screw_Terminal_01x02, TerminalBlock:TerminalBlock_MaiXu_MX126-5.0-02P_1x02_P5.00mm, symbol Connector:Screw_Terminal_01x02
- L2: footprint (none) -> Inductor_SMD:L_6.3x6.3_H3
- RFBB2, RFBT2: footprint (none) -> Resistor_SMD:R_0402_1005Metric
Connections:
- net +48V: now also J2.1 (Pin_1)
- net GND: now also J2.2 (Pin_2)
Other:
- moved on the sheet: U3

Commit message: update pcb routing:
Connections:
- net +5V: now reaches C14.1, CFF2.1, L2.2, RFBT2.1
- net +5V: now also U3.3 (VI)
- net +3.3V: now reaches U3.2 (VO)
Changed lines of the file:
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@@
 	(paper "A4")
-	(junction
-		(at 181.61 90.17)
-		(diameter 0)
-		(color 0 0 0 0)
-	)
 	(junction
 		(at 92.71 82.55)
@@
 	(junction
 		(at 107.95 85.09)
+		(diameter 0)
+		(color 0 0 0 0)
+	)
+	(junction
+		(at 181.61 90.17)
 		(diameter 0)
 		(color 0 0 0 0)
@@
 	)
 	(symbol
+		(lib_id "power:+5V")
+		(at 181.61 90.17 0)
+		(unit 1)
+		(body_style 1)
+		(exclude_from_sim no)
+		(in_bom yes)
+		(on_board yes)
+		(in_pos_files yes)
+		(dnp no)
+		(fields_autoplaced yes)
+		(property "Reference" "#PWR037"
+			(at 181.61 93.98 0)
+			(hide yes)
+			(show_name no)
+			(do_not_autoplace no)
+			(effects
+				(font
+					(size 1.27 1.27)
+				)
+			)
+		)
+		(property "Value" "+5V"
+			(at 181.61 85.09 0)
+			(show_name no)
+			(do_not_autoplace no)
+			(effects
+				(font
+					(size 1.27 1.27)
+				)
+			)
+		)
+		(property "Footprint" ""
+			(at 181.61 90.17 0)
+			(hide yes)
+			(show_name no)
+			(do_not_autoplace no)
+			(effects
+				(font
+					(size 1.27 1.27)
+				)
+			)
+		)
+		(property "Datasheet" ""
+			(at 181.61 90.17 0)
+			(hide yes)
+			(show_name no)
+			(do_not_autoplace no)
+			(effects
+				(font
+					(size 1.27 1.27)
+				)
+			)
+		)
+		(property "Description" "Power symbol creates a global label with name \"+5V\""
+			(at 181.61 90.17 0)
+			(hide yes)
+			(show_name no)
+			(do_not_autoplace no)
+			(effects
+				(font
+					(size 1.27 1.27)
+				)
+			)
+		)
+		(pin "1"
+		)
+		(instances
+			(project "ece-4275-final"
+				(path "/0c77f2af-cddb-472c-9a1b-8caed066380b/2b780b05-1c86-4b9a-ab1c-3f96b1a36c21"
+					(reference "#PWR037")
+					(unit 1)
+				)
+			)
+		)
+	)
+	(symbol
 		(lib_id "Device:C")
 		(at 92.71 86.36 0)
@@
 	)
 	(symbol
-		(lib_id "power:PWR_FLAG")
-		(at 140.97 59.69 0)
-		(unit 1)
-		(body_style 1)
-		(exclude_from_sim no)
-		(in_bom yes)
-		(on_board yes)
-		(in_pos_files yes)
-		(dnp no)
-		(fields_autoplaced yes)
-		(property "Reference" "#FLG02"
-			(at 140.97 57.785 0)
-			(hide yes)
-			(show_name no)
-			(do_not_autoplace no)
-			(effects
-				(font
-					(size 1.27 1.27)
-				)
-			)
-		)
-		(property "Value" "+5V"
-			(at 140.97 54.61 0)
-			(show_name no)
-			(do_not_autoplace no)
-			(effects
-				(font
-					(size 1.27 1.27)
-				)
-			)
-		)
-		(property "Footprint" ""
-			(at 140.97 59.69 0)
-			(hide yes)
-			(show_name no)
-			(do_not_autoplace no)
-			(effects
-				(font
-					(size 1.27 1.27)
-				)
-			)
-		)
-		(property "Datasheet" ""
-			(at 140.97 59.69 0)
-			(hide yes)
-			(show_name no)
-			(do_not_autoplace no)
-			(effects
-				(font
-					(size 1.27 1.27)
-				)
-			)
-		)
-		(property "Description" "Special symbol for telling ERC where power comes from"
-			(at 140.97 59.69 0)
-			(hide yes)
-			(show_name no)
-			(do_not_autoplace no)
-			(effects
-				(font
-					(size 1.27 1.27)
-				)
-			)
-		)
-		(pin "1"
-		)
-		(instances
-			(project "ece-4275-final"
-				(path "/0c77f2af-cddb-472c-9a1b-8caed066380b/2b780b05-1c86-4b9a-ab1c-3f96b1a36c21"
-					(reference "#FLG02")
-					(unit 1)
-				)
-			)
-		)
-	)
-	(symbol
 		(lib_id "Device:C")
 		(at 181.61 95.25 0)
@@
 	)
 	(symbol
-		(lib_id "power:PWR_FLAG")
+		(lib_id "power:+3.3V")
 		(at 156.21 59.69 0)
 		(unit 1)
@@
 		(dnp no)
 		(fields_autoplaced yes)
-		(property "Reference" "#FLG03"
-			(at 156.21 57.785 0)
+		(property "Reference" "#PWR035"
+			(at 156.21 63.5 0)
 			(hide yes)
 			(show_name no)
@@
 			)
 		)
-		(property "Description" "Special symbol for telling ERC where power comes from"
+		(property "Description" "Power symbol creates a global label with name \"+3.3V\""
 			(at 156.21 59.69 0)
 			(hide yes)
@@
 			(project "ece-4275-final"
 				(path "/0c77f2af-cddb-472c-9a1b-8caed066380b/2b780b05-1c86-4b9a-ab1c-3f96b1a36c21"
-					(reference "#FLG03")
+					(reference "#PWR035")
 					(unit 1)
 				)
@@
 	)
 	(symbol
+		(lib_id "power:+5V")
+		(at 140.97 59.69 0)
+		(unit 1)
+		(body_style 1)
+		(exclude_from_sim no)
+		(in_bom yes)
+		(on_board yes)
+		(in_pos_files yes)
+		(dnp no)
+		(fields_autoplaced yes)
+		(property "Reference" "#PWR036"
+			(at 140.97 63.5 0)
+			(hide yes)
+			(show_name no)
+			(do_not_autoplace no)
+			(effects
+				(font
+					(size 1.27 1.27)
+				)
+			)
+		)
+		(property "Value" "+5V"
+			(at 140.97 54.61 0)
+			(show_name no)
+			(do_not_autoplace no)
+			(effects
+				(font
+					(size 1.27 1.27)
+				)
+			)
+		)
+		(property "Footprint" ""
+			(at 140.97 59.69 0)
+			(hide yes)
+			(show_name no)
+			(do_not_autoplace no)
+			(effects
+				(font
+					(size 1.27 1.27)
+				)
+			)
+		)
+		(property "Datasheet" ""
+			(at 140.97 59.69 0)
+			(hide yes)
+			(show_name no)
+			(do_not_autoplace no)
+			(effects
+				(font
+					(size 1.27 1.27)
+				)
+			)
+		)
+		(property "Description" "Power symbol creates a global label with name \"+5V\""
+			(at 140.97 59.69 0)
+			(hide yes)
+			(show_name no)
+			(do_not_autoplace no)
+			(effects
+				(font
+					(size 1.27 1.27)
+				)
+			)
+		)
+		(pin "1"
+		)
+		(instances
+			(project "ece-4275-final"
+				(path "/0c77f2af-cddb-472c-9a1b-8caed066380b/2b780b05-1c86-4b9a-ab1c-3f96b1a36c21"
+					(reference "#PWR036")
+					(unit 1)
+				)
+			)
+		)
+	)
+	(symbol
 		(lib_id "IMPORTS:LMR36015ARNXR")
 		(at 130.81 97.79 0)
@@
 					(unit 1)
 				)
-			)
-		)
-	)
-	(symbol
-		(lib_id "power:PWR_FLAG")
-		(at 181.61 90.17 0)
-		(unit 1)
-		(body_style 1)
-		(exclude_from_sim no)
-		(in_bom yes)
-		(on_board yes)
-		(in_pos_files yes)
-		(dnp no)
-		(fields_autoplaced yes)
-		(property "Reference" "#FLG09"
-			(at 181.61 88.265 0)
-			(hide yes)
-			(show_name no)
-			(do_not_autoplace no)
-			(effects
-				(font
-					(size 1.27 1.27)
-				)
-			)
-		)
-		(property "Value" "+5V"
-			(at 181.61 85.09 0)
-			(show_name no)
-			(do_not_autoplace no)
-			(effects
-				(font
-					(size 1.27 1.27)
-				)
-			)
-		)
-		(property "Footprint" ""
-			(at 181.61 90.17 0)
-			(hide yes)
-			(show_name no)
-			(do_not_autoplace no)
-			(effects
-				(font
-					(size 1.27 1.27)
-				)
-			)
-		)
-		(property "Datasheet" ""
-			(at 181.61 90.17 0)
-			(hide yes)
-			(show_name no)
-			(do_not_autoplace no)
-			(effects
-				(font
-					(size 1.27 1.27)
-				)
-			)
-		)
-		(property "Description" "Special symbol for telling ERC where power comes from"
-			(at 181.61 90.17 0)
-			(hide yes)
-			(show_name no)
-			(do_not_autoplace no)
-			(effects
-				(font
-					(size 1.27 1.27)
-				)
-			)
-		)
-		(pin "1"
-		)
-		(instances
-			(project "ece-4275-final"
-				(path "/0c77f2af-cddb-472c-9a1b-8caed066380b/2b780b05-1c86-4b9a-ab1c-3f96b1a36c21"
-					(reference "#FLG09")
-					(unit 1)
-				)

Commit message: finish routing gpios
Parts:
- renumbered C13 to C17, C14 to C18, CBOOT2 to CBOOT1, CFF2 to CFF1, CHF3 to CHF1, CHF4 to CHF2, Cin2 to Cin1, J2 to J7, L2 to L1, RFBB2 to RFBB1, RFBT2 to RFBT1, U6 to U4, U3 to U5
Changed lines of the file:
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@@
 		(dnp no)
 		(fields_autoplaced yes)
-		(property "Reference" "#PWR015"
+		(property "Reference" "#PWR029"
 			(at 110.49 116.84 0)
 			(hide yes)
@@
 			(project "ece-4275-final"
 				(path "/0c77f2af-cddb-472c-9a1b-8caed066380b/2b780b05-1c86-4b9a-ab1c-3f96b1a36c21"
-					(reference "#PWR015")
+					(reference "#PWR029")
 					(unit 1)
 				)
@@
 		(dnp no)
 		(fields_autoplaced yes)
-		(property "Reference" "#PWR018"
+		(property "Reference" "#PWR035"
 			(at 172.72 116.84 0)
 			(hide yes)
@@
 			(project "ece-4275-final"
 				(path "/0c77f2af-cddb-472c-9a1b-8caed066380b/2b780b05-1c86-4b9a-ab1c-3f96b1a36c21"
-					(reference "#PWR018")
+					(reference "#PWR035")
 					(unit 1)
 				)
@@
 		(dnp no)
 		(fields_autoplaced yes)
-		(property "Reference" "L2"
+		(property "Reference" "L1"
 			(at 163.83 85.09 90)
 			(show_name no)
@@
 			(project "ece-4275-final"
 				(path "/0c77f2af-cddb-472c-9a1b-8caed066380b/2b780b05-1c86-4b9a-ab1c-3f96b1a36c21"
-					(reference "L2")
+					(reference "L1")
 					(unit 1)
 				)
@@
 		(dnp no)
 		(fields_autoplaced yes)
-		(property "Reference" "#PWR012"
+		(property "Reference" "#PWR025"
 			(at 92.71 96.52 0)
 			(hide yes)
@@
 			(project "ece-4275-final"
 				(path "/0c77f2af-cddb-472c-9a1b-8caed066380b/2b780b05-1c86-4b9a-ab1c-3f96b1a36c21"
-					(reference "#PWR012")
+					(reference "#PWR025")
 					(unit 1)
 				)
@@
 		(dnp no)
 		(fields_autoplaced yes)
-		(property "Reference" "#PWR037"
+		(property "Reference" "#PWR036"
 			(at 181.61 93.98 0)
 			(hide yes)
@@
 			(project "ece-4275-final"
 				(path "/0c77f2af-cddb-472c-9a1b-8caed066380b/2b780b05-1c86-4b9a-ab1c-3f96b1a36c21"
-					(reference "#PWR037")
+					(reference "#PWR036")
 					(unit 1)
 				)
@@
 		(dnp no)
 		(fields_autoplaced yes)
-		(property "Reference" "Cin2"
+		(property "Reference" "Cin1"
 			(at 96.52 85.0899 0)
 			(show_name no)
@@
 			(project "ece-4275-final"
 				(path "/0c77f2af-cddb-472c-9a1b-8caed066380b/2b780b05-1c86-4b9a-ab1c-3f96b1a36c21"
-					(reference "Cin2")
+					(reference "Cin1")
 					(unit 1)
 				)
@@
 		(in_pos_files yes)
 		(dnp no)
-		(property "Reference" "CBOOT2"
+		(property "Reference" "CBOOT1"
 			(at 156.21 74.93 90)
 			(show_name no)
@@
 			(project "ece-4275-final"
 				(path "/0c77f2af-cddb-472c-9a1b-8caed066380b/2b780b05-1c86-4b9a-ab1c-3f96b1a36c21"
-					(reference "CBOOT2")
+					(reference "CBOOT1")
 					(unit 1)
 				)
@@
 		(dnp no)
 		(fields_autoplaced yes)
-		(property "Reference" "#PWR027"
+		(property "Reference" "#PWR026"
 			(at 96.52 60.96 0)
 			(hide yes)
@@
 			(project "ece-4275-final"
 				(path "/0c77f2af-cddb-472c-9a1b-8caed066380b/2b780b05-1c86-4b9a-ab1c-3f96b1a36c21"
-					(reference "#PWR027")
+					(reference "#PWR026")
 					(unit 1)
 				)
@@
 		(dnp no)
 		(fields_autoplaced yes)
-		(property "Reference" "C14"
+		(property "Reference" "C18"
 			(at 185.42 93.9799 0)
 			(show_name no)
@@
 			(project "ece-4275-final"
 				(path "/0c77f2af-cddb-472c-9a1b-8caed066380b/2b780b05-1c86-4b9a-ab1c-3f96b1a36c21"
-					(reference "C14")
+					(reference "C18")
 					(unit 1)
 				)
@@
 		(dnp no)
 		(fields_autoplaced yes)
-		(property "Reference" "CHF3"
+		(property "Reference" "CHF1"
 			(at 80.01 85.0899 0)
 			(show_name no)
@@
 			(project "ece-4275-final"
 				(path "/0c77f2af-cddb-472c-9a1b-8caed066380b/2b780b05-1c86-4b9a-ab1c-3f96b1a36c21"
-					(reference "CHF3")
+					(reference "CHF1")
 					(unit 1)
 				)
@@
 		(dnp no)
 		(fields_autoplaced yes)
-		(property "Reference" "J2"
+		(property "Reference" "J7"
 			(at 99.06 60.9599 90)
 			(show_name no)
@@
 			(project "ece-4275-final"
 				(path "/0c77f2af-cddb-472c-9a1b-8caed066380b/2b780b05-1c86-4b9a-ab1c-3f96b1a36c21"
-					(reference "J2")
+					(reference "J7")
 					(unit 1)
 				)
@@
 		(dnp no)
 		(fields_autoplaced yes)
-		(property "Reference" "#PWR028"
+		(property "Reference" "#PWR024"
 			(at 90.17 66.04 0)
 			(hide yes)
@@
 			(project "ece-4275-final"
 				(path "/0c77f2af-cddb-472c-9a1b-8caed066380b/2b780b05-1c86-4b9a-ab1c-3f96b1a36c21"
-					(reference "#PWR028")
+					(reference "#PWR024")
 					(unit 1)
 				)
@@
 		(dnp no)
 		(fields_autoplaced yes)
-		(property "Reference" "CHF4"
+		(property "Reference" "CHF2"
 			(at 87.63 85.0899 0)
 			(show_name no)
@@
 			(project "ece-4275-final"
 				(path "/0c77f2af-cddb-472c-9a1b-8caed066380b/2b780b05-1c86-4b9a-ab1c-3f96b1a36c21"
-					(reference "CHF4")
+					(reference "CHF2")
 					(unit 1)
 				)
@@
 		(dnp no)
 		(fields_autoplaced yes)
-		(property "Reference" "#PWR035"
+		(property "Reference" "#PWR034"
 			(at 156.21 63.5 0)
 			(hide yes)
@@
 			(project "ece-4275-final"
 				(path "/0c77f2af-cddb-472c-9a1b-8caed066380b/2b780b05-1c86-4b9a-ab1c-3f96b1a36c21"
-					(reference "#PWR035")
+					(reference "#PWR034")
 					(unit 1)
 				)
@@
 		(dnp no)
 		(fields_autoplaced yes)
-		(property "Reference" "U3"
+		(property "Reference" "U5"
 			(at 148.59 53.34 0)
 			(show_name no)
@@
 			(project "ece-4275-final"
 				(path "/0c77f2af-cddb-472c-9a1b-8caed066380b/2b780b05-1c86-4b9a-ab1c-3f96b1a36c21"
-					(reference "U3")
+					(reference "U5")
 					(unit 1)
 				)
@@
 		(dnp no)
 		(fields_autoplaced yes)
-		(property "Reference" "#PWR016"
+		(property "Reference" "#PWR032"
 			(at 152.4 104.14 0)
 			(hide yes)
@@
 			(project "ece-4275-final"
 				(path "/0c77f2af-cddb-472c-9a1b-8caed066380b/2b780b05-1c86-4b9a-ab1c-3f96b1a36c21"
-					(reference "#PWR016")
+					(reference "#PWR032")
 					(unit 1)
 				)
@@
 		(dnp no)
 		(fields_autoplaced yes)
-		(property "Reference" "#PWR036"
+		(property "Reference" "#PWR030"
 			(at 140.97 63.5 0)
 			(hide yes)
@@
 			(project "ece-4275-final"
 				(path "/0c77f2af-cddb-472c-9a1b-8caed066380b/2b780b05-1c86-4b9a-ab1c-3f96b1a36c21"
-					(reference "#PWR036")
+					(reference "#PWR030")
 					(unit 1)
 				)
@@
 		(dnp no)
 		(fields_autoplaced yes)
-		(property "Reference" "U6"
+		(property "Reference" "U4"
 			(at 130.81 72.39 0)
 			(show_name no)
@@
 			(project "ece-4275-final"
 				(path "/0c77f2af-cddb-472c-9a1b-8caed066380b/2b780b05-1c86-4b9a-ab1c-3f96b1a36c21"
-					(reference "U6")
+					(reference "U4")
 					(unit 1)
 				)
@@
 		(dnp no)
 		(fields_autoplaced yes)
-		(property "Reference" "RFBT2"
+		(property "Reference" "RFBT1"
 			(at 174.5635 97.7899 0)
 			(show_name no)
@@
 			(project "ece-4275-final"
 				(path "/0c77f2af-cddb-472c-9a1b-8caed066380b/2b780b05-1c86-4b9a-ab1c-3f96b1a36c21"
-					(reference "RFBT2")
+					(reference "RFBT1")
 					(unit 1)
 				)
@@
 		(dnp no)
 		(fields_autoplaced yes)
-		(property "Reference" "#PWR019"
+		(property "Reference" "#PWR037"
 			(at 181.61 105.41 0)
 			(hide yes)
@@
 			(project "ece-4275-final"
 				(path "/0c77f2af-cddb-472c-9a1b-8caed066380b/2b780b05-1c86-4b9a-ab1c-3f96b1a36c21"
-					(reference "#PWR019")
+					(reference "#PWR037")
 					(unit 1)
 				)
@@
 		(dnp no)
 		(fields_autoplaced yes)
-		(property "Reference" "#PWR014"
+		(property "Reference" "#PWR028"
 			(at 107.95 80.01 0)
 			(hide yes)
@@
 			(project "ece-4275-final"
 				(path "/0c77f2af-cddb-472c-9a1b-8caed066380b/2b780b05-1c86-4b9a-ab1c-3f96b1a36c21"
-					(reference "#PWR014")
+					(reference "#PWR028")
 					(unit 1)
 				)
@@
 		(in_pos_files yes)
 		(dnp no)
-		(property "Reference" "CFF2"
+		(property "Reference" "CFF1"
 			(at 166.878 97.028 0)
 			(show_name no)
@@
 			(project "ece-4275-final"
 				(path "/0c77f2af-cddb-472c-9a1b-8caed066380b/2b780b05-1c86-4b9a-ab1c-3f96b1a36c21"
-					(reference "CFF2")
+					(reference "CFF1")
 					(unit 1)
 				)
@@
 		(dnp no)
 		(fields_autoplaced yes)
-		(property "Reference" "#PWR010"
+		(property "Reference" "#PWR031"
 			(at 148.59 73.66 0)
 			(hide yes)
@@
 			(project "ece-4275-final"
 				(path "/0c77f2af-cddb-472c-9a1b-8caed066380b/2b780b05-1c86-4b9a-ab1c-3f96b1a36c21"
-					(reference "#PWR010")
+					(reference "#PWR031")
 					(unit 1)
 				)
@@
 		(dnp no)
 		(fields_autoplaced yes)
-		(property "Reference" "#PWR013"
+		(property "Reference" "#PWR027"
 			(at 105.41 104.14 0)
 			(hide yes)
@@
 			(project "ece-4275-final"
 				(path "/0c77f2af-cddb-472c-9a1b-8caed066380b/2b780b05-1c86-4b9a-ab1c-3f96b1a36c21"
-					(reference "#PWR013")
+					(reference "#PWR027")
 					(unit 1)
 				)
@@
 		(dnp no)
 		(fields_autoplaced yes)
-		(property "Reference" "C13"
+		(property "Reference" "C17"
 			(at 114.3 105.4099 0)
 			(show_name no)
@@
 			(project "ece-4275-final"
 				(path "/0c77f2af-cddb-472c-9a1b-8caed066380b/2b780b05-1c86-4b9a-ab1c-3f96b1a36c21"
-					(reference "C13")
+					(reference "C17")
 					(unit 1)
 				)
@@
 		(dnp no)
 		(fields_autoplaced yes)
-		(property "Reference" "#PWR017"
+		(property "Reference" "#PWR033"
 			(at 152.4 119.38 0)
 			(hide yes)
@@
 			(project "ece-4275-final"
 				(path "/0c77f2af-cddb-472c-9a1b-8caed066380b/2b780b05-1c86-4b9a-ab1c-3f96b1a36c21"
-					(reference "#PWR017")
+					(reference "#PWR033")
 					(unit 1)
 				)
@@
 		(dnp no)
 		(fields_autoplaced yes)
-		(property "Reference" "RFBB2"
+		(property "Reference" "RFBB1"
 			(at 174.5635 105.4099 0)
 			(show_name no)
@@
 			(project "ece-4275-final"
 				(path "/0c77f2af-cddb-472c-9a1b-8caed066380b/2b780b05-1c86-4b9a-ab1c-3f96b1a36c21"
-					(reference "RFBB2")
-					(unit 1)
-				)
+					(reference "RFBB1")
+					(unit 1)
+				)
