File: kicad/ece-4275-final.kicad_pcb (KiCad board)
At the start: 2 copper layers, 96.5 x 63.5 mm, 68 parts, among them J1 USB_C_Receptacle_USB2.0_14P, J2 Screw_Terminal_01x02, J3 Conn_01x08, J4 Conn_01x08, J5 Conn_01x02, J6 STEPPER_1_JST_XH, Q1 BSZ150N10LS3-G, Q2 BSZ150N10LS3-G, Q3 BSZ150N10LS3-G, Q4 BSZ150N10LS3-G, Q5 BSZ150N10LS3-G, Q6 BSZ150N10LS3-G, Q7 BSZ150N10LS3-G, Q8 BSZ150N10LS3-G, Q9 AO3400A, U1 ESP32-S3-WROOM-1, U2 USBLC6-2SC6, U3 AMS1117-3.3, U5 TMC5160A-TA, U6 LMR36015ARNXR

Commit message: finish routing gpios
Parts:
- removed the J5 at (194.1, 106.6)
- removed RFBT2: 52.3k, Resistor_SMD:R_0402_1005Metric
- added C22: 100nF, Capacitor_SMD:C_0402_1005Metric, F.Cu at (159.1, 80.9)
- added C23: 100nF, Capacitor_SMD:C_0402_1005Metric, F.Cu at (151.9, 80.9)
- added C24: 100nF, Capacitor_SMD:C_0402_1005Metric, F.Cu at (144.7, 80.9)
- added J1: LED_CONN_1, Connector_JST:JST_PH_B3B-PH-K_1x03_P2.00mm_Vertical, F.Cu at (175.2, 70.3)
- added J14: LIMIT_0, Connector_JST:JST_PH_B2B-PH-K_1x02_P2.00mm_Vertical, F.Cu at (157.6, 77.1)
- added J15: LIMIT_1, Connector_JST:JST_PH_B2B-PH-K_1x02_P2.00mm_Vertical, F.Cu at (150.4, 77.1)
- added J16: LIMIT_2, Connector_JST:JST_PH_B2B-PH-K_1x02_P2.00mm_Vertical, F.Cu at (143.2, 77.1)
- added J2: LED_CONN_0, Connector_JST:JST_PH_B3B-PH-K_1x03_P2.00mm_Vertical, F.Cu at (175.2, 59.1)
- added JFAN0: FAN, Connector_JST:JST_PH_B2B-PH-K_1x02_P2.00mm_Vertical, F.Cu at (156.7, 89.8)
- added JFAN1: FAN, Connector_JST:JST_PH_B2B-PH-K_1x02_P2.00mm_Vertical, F.Cu at (149.7, 89.8)
- added JFAN2: FAN, Connector_JST:JST_PH_B2B-PH-K_1x02_P2.00mm_Vertical, F.Cu at (142.7, 89.8)
- added Q10: AO3400A, Package_TO_SOT_SMD:SOT-23, F.Cu at (146.2, 84.3)
- added Q11: AO3400A, Package_TO_SOT_SMD:SOT-23, F.Cu at (142.4, 84.2)
- added R2: 330, Resistor_SMD:R_0402_1005Metric, F.Cu at (171.9, 59.1)
- added R21: 330, Resistor_SMD:R_0402_1005Metric, F.Cu at (172.0, 70.3)
- added REF**: MountingHole_3.2mm_M3, MountingHole:MountingHole_3.2mm_M3, F.Cu at (104.1, 107.5)
- added REF**: MountingHole_3.2mm_M3, MountingHole:MountingHole_3.2mm_M3, F.Cu at (104.0, 52.0)
- added REF**: MountingHole_3.2mm_M3, MountingHole:MountingHole_3.2mm_M3, F.Cu at (192.5, 107.5)
- added REF**: MountingHole_3.2mm_M3, MountingHole:MountingHole_3.2mm_M3, F.Cu at (192.5, 52.0)
- J3: value Conn_01x08 -> TX_RX; footprint Connector_PinHeader_2.54mm:PinHeader_1x08_P2.54mm_Vertical -> Connector_JST:JST_PH_B2B-PH-K_1x02_P2.00mm_Vertical
- J4: value Conn_01x08 -> GPIO_38_48; footprint Connector_PinHeader_2.54mm:PinHeader_1x08_P2.54mm_Vertical -> Connector_PinHeader_2.54mm:PinHeader_1x09_P2.54mm_Vertical
- moved J4 94.4 mm to (164.4, 73.4), turned to 180 degrees
- moved BOOT1 94.2 mm to (159.9, 70.6), turned to -90 degrees
- moved EN1 68.0 mm to (133.0, 57.8), turned to 90 degrees
- moved RFBB1 58.3 mm to (129.0, 97.4), turned to 180 degrees
- moved R15 56.6 mm to (104.6, 84.3)
- moved J3 39.7 mm to (169.9, 53.7), turned to -90 degrees
- moved Q9 38.8 mm to (149.8, 84.3), turned to -90 degrees
- moved R1 28.5 mm to (158.5, 66.3)
- moved R4 20.6 mm to (111.8, 53.1), turned to 90 degrees
- moved R5 11.4 mm to (123.5, 53.0), turned to -90 degrees
- moved R3 6.23 mm to (137.1, 52.5), turned to -90 degrees
- moved C18 5.00 mm to (131.5, 99.0)
- moved Cin1 4.79 mm to (136.7, 98.3)
- moved CHF1 4.09 mm to (134.5, 98.3)
- moved CHF2 4.04 mm to (135.6, 98.3)
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- renumbered C9 to C1, C18 to C10, C19 to C11, C5 to C12, C1 to C13, C3 to C14, C7 to C15, C20 to C16, C13 to C17, C14 to C18, C10 to C2, C2 to C3, C6 to C5, C15 to C6, C8 to C7, C17 to C8, C16 to C9, CBOOT2 to CBOOT1, CFF2 to CFF1, CHF3 to CHF1, CHF4 to CHF2, Cin2 to Cin1, J1 to J5, J2 to J7, L2 to L1, R17 to R1, R7 to R10, R8 to R11, R9 to R12, R10 to R15, R4 to R16, R5 to R17, R15 to R18, R11 to R19, R12 to R20, R16 to R3, R18 to R4, R19 to R5, R1 to R6, R2 to R7, R3 to R8, R6 to R9, RFBB2 to RFBB1, U5 to U3, U6 to U4, U3 to U5
Connections:
- J3 pad 1: GND -> Net-(J3-Pin_1)
- J3 pad 2: GND -> Net-(J3-Pin_2)
- J4 pad 1: unconnected-(J4-Pin_1-Pad1) -> Net-(J4-Pin_1)
- J4 pad 2: unconnected-(J4-Pin_2-Pad2) -> Net-(J4-Pin_2)
- J4 pad 3: unconnected-(J4-Pin_3-Pad3) -> Net-(J4-Pin_3)
- J4 pad 4: unconnected-(J4-Pin_4-Pad4) -> Net-(J4-Pin_4)
- J4 pad 5: unconnected-(J4-Pin_5-Pad5) -> Net-(J4-Pin_5)
- J4 pad 6: unconnected-(J4-Pin_6-Pad6) -> Net-(J4-Pin_6)
- J4 pad 7: unconnected-(J4-Pin_7-Pad7) -> Net-(J4-Pin_7)
- J4 pad 8: unconnected-(J4-Pin_8-Pad8) -> Net-(J4-Pin_8)
- Q9 pad 1: unconnected-(Q9-G-Pad1) -> /Two Pin Fan/IN
- U1 pad 12: unconnected-(U1-IO8-Pad12) -> /Two Pin Fan2/IN
- U1 pad 16: unconnected-(U1-IO46-Pad16) -> Net-(J4-Pin_7)
- U1 pad 17: unconnected-(U1-IO9-Pad17) -> /Two Pin Fan1/IN
- U1 pad 18: unconnected-(U1-IO10-Pad18) -> /Two Pin Fan/IN
- U1 pad 24: unconnected-(U1-IO47-Pad24) -> Net-(J4-Pin_8)
- U1 pad 25: unconnected-(U1-IO48-Pad25) -> Net-(J4-Pin_9)
- U1 pad 26: unconnected-(U1-IO45-Pad26) -> Net-(J4-Pin_6)
- U1 pad 31: unconnected-(U1-IO38-Pad31) -> Net-(J4-Pin_1)
- U1 pad 32: unconnected-(U1-IO39-Pad32) -> Net-(J4-Pin_2)
- U1 pad 33: unconnected-(U1-IO40-Pad33) -> Net-(J4-Pin_3)
- U1 pad 34: unconnected-(U1-IO41-Pad34) -> Net-(J4-Pin_4)
- U1 pad 35: unconnected-(U1-IO42-Pad35) -> Net-(J4-Pin_5)
- U1 pad 36: unconnected-(U1-RXD0-Pad36) -> Net-(J3-Pin_2)
- U1 pad 37: unconnected-(U1-TXD0-Pad37) -> Net-(J3-Pin_1)
- U1 pad 38: unconnected-(U1-IO2-Pad38) -> /LIMIT_1
- U1 pad 39: unconnected-(U1-IO1-Pad39) -> /LIMIT_0
- U1 pad 4: unconnected-(U1-IO4-Pad4) -> /LIMIT_2
- U1 pad 6: unconnected-(U1-IO6-Pad6) -> Net-(U1-IO6)
- U1 pad 7: unconnected-(U1-IO7-Pad7) -> Net-(U1-IO7)
Routing:
- net +5V: track 51.2 -> 199.3 mm, vias 0 -> 5
- net Net-(U1-IO7): track 0.00 -> 45.6 mm, vias 0 -> 2
- net Net-(U1-IO6): track 0.00 -> 43.5 mm
- net +3.3V: track 68.6 -> 110.6 mm, vias 2 -> 7
- net GND: track 42.9 -> 84.2 mm, vias 14 -> 17
- net /LIMIT_0: track 0.00 -> 37.5 mm, vias 0 -> 2
- net Net-(J4-Pin_7): track 0.00 -> 37.2 mm, vias 0 -> 1
- net /LIMIT_1: track 0.00 -> 30.6 mm, vias 0 -> 2
- net /LIMIT_2: track 0.00 -> 30.6 mm, vias 0 -> 2
- net /Two Pin Fan2/IN: track 0.00 -> 21.8 mm, vias 0 -> 2
- net Net-(Q5-G): track 0.00 -> 19.7 mm, vias 0 -> 2
- net Net-(J4-Pin_9): track 0.00 -> 19.1 mm, vias 0 -> 1
- net /Two Pin Fan/IN: track 0.00 -> 18.5 mm, vias 0 -> 2
- net Net-(J4-Pin_8): track 0.00 -> 18.1 mm, vias 0 -> 1
- net /Two Pin Fan1/IN: track 0.00 -> 17.8 mm, vias 0 -> 2
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Other:
- board text added: "D38"
- board text added: "D39"
- board text added: "D40"
- board text added: "D41"
- board text added: "D42"
- board text added: "D45"
- board text added: "D46"
- board text added: "D47"
- board text added: "D48"
- board text added: "USB-C"

Commit message: final?
Parts:
- added C19: 0.1uF, Capacitor_SMD:C_0402_1005Metric, F.Cu at (166.5, 88.6)
- added C20: 0.1uF, Capacitor_SMD:C_0402_1005Metric, F.Cu at (166.5, 92.9)
- added POWER_LED1: LED, LED_THT:LED_D10.0mm, F.Cu at (168.8, 102.5)
- added R22: 10k, Resistor_SMD:R_0402_1005Metric, F.Cu at (166.5, 87.4)
- added R23: 10k, Resistor_SMD:R_0402_1005Metric, F.Cu at (166.5, 94.0)
- added R24: 680, Resistor_SMD:R_0402_1005Metric, F.Cu at (163.9, 110.1)
- added RFBT1: 52.3k, Resistor_SMD:R_0402_1005Metric, F.Cu at (133.5, 99.0)
- added THERM1: THERM1, Connector_JST:JST_PH_B2B-PH-K_1x02_P2.00mm_Vertical, F.Cu at (170.2, 87.4)
- added THERM2: THERM2, Connector_JST:JST_PH_B2B-PH-K_1x02_P2.00mm_Vertical, F.Cu at (170.2, 94.0)
- moved R20 1.60 mm to (108.1, 67.4)
- moved C5 0.08 mm to (118.5, 73.9)
Connections:
- U1 pad 10: unconnected-(U1-IO17-Pad10) -> /LIMIT_2
- U1 pad 11: unconnected-(U1-IO18-Pad11) -> /DRV_1_DIR
- U1 pad 4: /LIMIT_2 -> Net-(U1-IO4)
- U1 pad 5: unconnected-(U1-IO5-Pad5) -> Net-(U1-IO5)
- U1 pad 8: unconnected-(U1-IO15-Pad8) -> /DRV_1_CS
- U1 pad 9: unconnected-(U1-IO16-Pad9) -> /DRV_1_STEP
Routing:
- net +3.3V: track 110.6 -> 172.0 mm, vias 7 -> 6
- net Net-(U1-IO5): track 0.00 -> 50.6 mm, vias 0 -> 2
- net Net-(U1-IO4): track 0.00 -> 48.6 mm, vias 0 -> 2
- net Net-(Q3-G): track 0.00 -> 33.3 mm, vias 0 -> 2
- net +48V: track 132.5 -> 161.8 mm
- net Net-(Q1-G): track 0.00 -> 28.6 mm, vias 0 -> 2
- net /DRV_1_CS: track 0.00 -> 27.5 mm, vias 0 -> 2
- net Net-(Q4-D): track 30.1 -> 55.8 mm, vias 2 -> 3
- net /DRV_1_STEP: track 0.00 -> 21.2 mm
- net /DRV_1_DIR: track 0.00 -> 20.0 mm, vias 0 -> 2
- net GND: track 84.2 -> 102.6 mm, vias 17 -> 18
- net Net-(U3-VCC): track 3.26 -> 21.2 mm, vias 0 -> 2
- net Net-(Q7-G): track 0.00 -> 17.1 mm, vias 0 -> 2
- net Net-(POWER_LED1-A): track 0.00 -> 6.92 mm
- net /LIMIT_2: track 30.6 -> 25.3 mm
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Other:
- board text added: "ESP32-S3 GPIO MAP ----------- GPIO1 LIMIT0 GPIO2 LIMIT1 GPIO17 LIMIT2 GPIO8 FAN2 GPIO9 FAN1 GPIO10 FAN0 GPIO11 DRV MOSI GPIO12 DRV SCK GPIO13 DRV MISO GPIO14 DRV ENA GPIO15 DRV CS GPIO16 DRV STEP GPIO18 DRV DIR GPIO38 J4.1 GPIO39 J4.2 GPIO40 J4.3 GPIO41 J4.4 GPIO42 J4.5 GPIO45 J4.6 GPIO46 J4.7 GPIO47 J4.8 GPIO48 J4.9 GPIO43 TX0 (J3.1) GPIO44 RX0 (J3.2) GPIO19 USB- GPIO20 USB+"
