File: kicad/stepper_module.kicad_sch (KiCad schematic)
At the start: 7 parts, among them U5 TMC5160A-TA

Commit message: finish motor driver module
Parts:
- added C1, C3, C5, C7: CB, symbol Device:C
- added C17, C18: 100nF, symbol Device:C
- added C19, C20: 470nF, symbol Device:C
- added C8: 22n, 100V, symbol Device:C
- added C_E1: C_Polarized, symbol Device:C_Polarized
- added Q1, Q2, Q3, Q4, Q5, Q6, Q7, Q8: BSC440N10NS3G, Package_TO_SOT_SMD:TDSON-8-1, symbol Transistor_FET:BSC440N10NS3G
- added R10, R15: RS, symbol Device:R
- added R11, R12, R2, R3, R4, R5, R6, R7: RG, symbol Device:R
- added R13, R14, R8, R9: 47, symbol Device:R
- renumbered R to R1
Connections:
- net +48V: now also U5.33 (VS), C17.2, C18.2, C19.2, C20.2, C_E1.1, Q1.5 (D), Q3.1 (S), Q3.2 (S), Q3.3 (S)
- net GND: now also C18.1, C20.1, C_E1.2, R10.1, R14.2, R15.1, R9.2
- net at U5.1 (HB1): now also R6.1
- net at U5.10 (SRBL): now also R14.1
- net TST_MODE: now reaches U5.11 (TST_MODE)
- net REFL_STEP: now reaches U5.17 (REFL/STEP)
- net REFL_DIR: now reaches U5.18 (REFR/DIR)
- net at U5.2 (CB1): now also C3.1
- net SD_MODE: now reaches U5.21 (SD_MODE)
- net SPI_MODE: now reaches U5.22 (SPI_MODE)
- net ENC_B_DCEN: now reaches U5.23 (ENCB/DCEN/CFG4)
- net ENC_A_DCIN: now reaches U5.24 (ENCA/DCIN/CFG5)
- net ENC_N_DCO: now reaches U5.25 (ENCN/DCO/CFG6)
- net DIAG0_SWN: now reaches U5.26 (SWN/DIAG0)
- net DIAG1_SWP: now reaches U5.27 (SWP/DIAG1)
- net at U5.31 (CPO): now also C8.1
- net at U5.32 (CPI): now also C8.2
- net at U5.34 (VCP): now also C17.1
- net at U5.35 (CA2): now also C7.2
- net at U5.36 (HA2): now also R4.2
- net A2: now reaches U5.37 (BMA2)
- net A2: now also C7.1, Q2.4 (G), Q3.5 (D), Q4.1 (S), Q4.2 (S), Q4.3 (S), R3.2
- net at U5.38 (LA2): now also R5.2
- net at U5.39 (LA1): now also R3.1
- net A1: now reaches U5.40 (BMA1)
- net A1: now also C5.1, Q1.1 (S), Q1.2 (S), Q1.3 (S), Q2.5 (D)
- net at U5.41 (HA1): now also R2.1
- net at U5.42 (CA1): now also C5.2
- net at U5.43 (CB2): now also C1.1
- net at U5.44 (HB2): now also R11.1
- net B2: now reaches U5.45 (BMB2)
- net B2: now also C1.2, Q7.5 (D), Q8.1 (S), Q8.2 (S), Q8.3 (S)
- net at U5.46 (LB2): now also Q2.1 (S), Q2.2 (S), Q2.3 (S), Q4.5 (D), R10.2, R12.1, R8.2
- net at U5.47 (LB1): now also R7.1
- net B1: now reaches U5.48 (BMB1)
- net B1: now also C3.2, Q5.1 (S), Q5.2 (S), Q5.3 (S), Q6.5 (D)
- net at U5.7 (SRAL): now also R9.1
- net at U5.8 (SRAH): now also R8.1
- net at U5.9 (SRBH): now also R13.1
- new net: Q6.4 (G), R7.2
- new net: Q3.4 (G), R4.1
- new net: R13.2, R15.2
- new net: Q1.4 (G), R2.2
- new net: Q5.5 (D), Q7.1 (S), Q7.2 (S), Q7.3 (S)
- new net: Q7.4 (G), R11.2
- new net: Q5.4 (G), R6.2
- new net: Q8.4 (G), R12.2
- new net: Q6.1 (S), Q6.2 (S), Q6.3 (S), Q8.5 (D)
- new net: Q4.4 (G), R5.1

Commit message: edit a lot of stuff
Parts:
- C1, C15, C16, C17, C18, C19, C2, C20, C3, C4, C5, C6, C7, C8: footprint (none) -> Capacitor_SMD:C_0402_1005Metric
- C_E1: footprint (none) -> Capacitor_SMD:CP_Elec_3x5.3
- Q1, Q2, Q3, Q4, Q5, Q6, Q7, Q8: value BSC440N10NS3G -> BSZ150N10NS3-G; footprint Package_TO_SOT_SMD:TDSON-8-1 -> Package_SON:VSON-8_3.3x3.3mm_P0.65mm_NexFET
- R1, R10, R11, R12, R13, R14, R15, R2, R3, R4, R5, R6, R7, R8, R9: footprint (none) -> Resistor_SMD:R_0402_1005Metric

Commit message: update pcb routing:
Parts:
- Q1, Q2, Q3, Q4, Q5, Q6, Q7, Q8: value BSZ150N10NS3-G -> BSZ150N10LS3-G
Connections:
- net GND: now also C19.1
Changed lines of the file:
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@@
 	)
 	(junction
+		(at 96.52 27.94)
+		(diameter 0)
+		(color 0 0 0 0)
+	)
+	(junction
 		(at 43.18 27.94)
 		(diameter 0)
@@
 	(wire
 		(pts
+			(xy 96.52 27.94) (xy 102.87 27.94)
+		)
+		(stroke
+			(width 0)
+			(type default)
+		)
+	)
+	(wire
+		(pts
 			(xy 105.41 85.09) (xy 133.35 85.09)
 		)
@@
 			)
 		)
-		(property "Value" "BSZ150N10NS3-G"
+		(property "Value" "BSZ150N10LS3-G"
 			(at 158.75 43.942 0)
 			(show_name no)
@@
 			)
 		)
-		(property "Value" "BSZ150N10NS3-G"
+		(property "Value" "BSZ150N10LS3-G"
 			(at 177.8 69.088 0)
 			(show_name no)
@@
 			)
 		)
-		(property "Value" "BSZ150N10NS3-G"
+		(property "Value" "BSZ150N10LS3-G"
 			(at 177.8 79.248 0)
 			(show_name no)
@@
 			)
 		)
-		(property "Value" "BSZ150N10NS3-G"
+		(property "Value" "BSZ150N10LS3-G"
 			(at 132.08 39.878 0)
 			(show_name no)
@@
 			)
 		)
-		(property "Value" "BSZ150N10NS3-G"
+		(property "Value" "BSZ150N10LS3-G"
 			(at 158.75 33.782 0)
 			(show_name no)
@@
 			)
 		)
-		(property "Value" "BSZ150N10NS3-G"
+		(property "Value" "BSZ150N10LS3-G"
 			(at 132.08 50.038 0)
 			(show_name no)
@@
 			)
 		)
-		(property "Value" "BSZ150N10NS3-G"
+		(property "Value" "BSZ150N10LS3-G"
 			(at 204.47 73.152 0)
 			(show_name no)
@@
 			)
 		)
-		(property "Value" "BSZ150N10NS3-G"
+		(property "Value" "BSZ150N10LS3-G"
 			(at 204.47 62.992 0)
 			(show_name no)

Commit message: finish routing gpios
Parts:
- renumbered C18 to C10, C19 to C11, C5 to C12, C1 to C13, C3 to C14, C7 to C15, C20 to C16, C2 to C3, C6 to C5, C15 to C6, C8 to C7, C17 to C8, C16 to C9, R7 to R10, R8 to R11, R9 to R12, R10 to R15, R4 to R16, R5 to R17, R15 to R18, R11 to R19, R12 to R20, R1 to R6, R2 to R7, R3 to R8, R6 to R9, U5 to U3

Commit message: final?
Parts:
- C12, C13, C14, C15: value CB -> 220nF
- R10, R16, R17, R19, R20, R7, R8, R9: value RG -> 22
- R15, R18: value RS -> 100m
- R6: value 2R2 -> 2.2
Changed lines of the file:
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@@
 			)
 		)
-		(property "Value" "RG"
+		(property "Value" "22"
 			(at 110.236 57.912 90)
 			(show_name no)
@@
 			)
 		)
-		(property "Value" "RG"
+		(property "Value" "22"
 			(at 172.466 37.592 90)
 			(show_name no)
@@
 			)
 		)
-		(property "Value" "RS"
+		(property "Value" "100m"
 			(at 189.484 90.17 90)
 			(show_name no)
@@
 			)
 		)
-		(property "Value" "CB"
+		(property "Value" "220nF"
 			(at 128.524 80.772 90)
 			(show_name no)
@@
 			)
 		)
-		(property "Value" "RG"
+		(property "Value" "22"
 			(at 110.236 52.832 90)
 			(show_name no)
@@
 			)
 		)
-		(property "Value" "RG"
+		(property "Value" "22"
 			(at 110.236 42.164 90)
 			(show_name no)
@@
 			)
 		)
-		(property "Value" "RS"
+		(property "Value" "100m"
 			(at 143.764 68.58 90)
 			(show_name no)
@@
 			)
 		)
-		(property "Value" "RG"
+		(property "Value" "22"
 			(at 199.136 84.582 90)
 			(show_name no)
@@
 			)
 		)
-		(property "Value" "CB"
+		(property "Value" "220nF"
 			(at 139.446 84.328 90)
 			(show_name no)
@@
 			)
 		)
-		(property "Value" "RG"
+		(property "Value" "22"
 			(at 197.866 59.182 90)
 			(show_name no)
@@
 			)
 		)
-		(property "Value" "CB"
+		(property "Value" "220nF"
 			(at 133.096 86.868 90)
 			(show_name no)
@@
 			)
 		)
-		(property "Value" "RG"
+		(property "Value" "22"
 			(at 110.236 37.592 90)
 			(show_name no)
@@
 			)
 		)
-		(property "Value" "CB"
+		(property "Value" "220nF"
 			(at 142.494 83.312 90)
 			(show_name no)
@@
 			)
 		)
-		(property "Value" "RG"
+		(property "Value" "22"
 			(at 172.466 47.752 90)
 			(show_name no)
@@
 			)
 		)
-		(property "Value" "2R2"
+		(property "Value" "2.2"
 			(at 55.88 30.4799 0)
 			(show_name no)
